File: electronics/occulink-quad-sata.kicad_pcb (KiCad board)
At the start: 4 copper layers, 5 parts, among them P0 MOLEX_NANOPITCH_42_WAY, P1 MOLEX_SATA_COMBO, P2 MOLEX_SATA_COMBO, P3 MOLEX_SATA_COMBO, P4 MOLEX_SATA_COMBO

Commit message: PCB layout tests
Parts:
- added C1: 10u_X7S_3225M, Applidyne_Capacitor:CAPC3225X170N, B.Cu at (134.0, 105.8)
- added C2: 10u_X7S_3225M, Applidyne_Capacitor:CAPC3225X170N, B.Cu at (134.0, 116.0)
- added C3: 10u_X7S_3225M, Applidyne_Capacitor:CAPC3225X170N, B.Cu at (134.0, 126.0)
- added C5: 10u_X7S_3225M, Applidyne_Capacitor:CAPC3225X170N, B.Cu at (129.0, 105.8)
- added C6: 10u_X7S_3225M, Applidyne_Capacitor:CAPC3225X170N, B.Cu at (129.0, 116.0)
- added C7: 10u_X7S_3225M, Applidyne_Capacitor:CAPC3225X170N, B.Cu at (129.0, 126.0)
- added P5: MOLEX_MINIFIT_JR_2x2_WAY, Applidyne_Connector_Molex:Molex_Mini-Fit_Jr_5566-04A_2x02_P4.20mm_Vertical, B.Cu at (94.5, 130.0)
- added R1: 0R_1608M, Applidyne_Resistor:RESC1608X50N, B.Cu at (139.2, 105.2)
- added R2: 0R_1608M, Applidyne_Resistor:RESC1608X50N, B.Cu at (139.2, 106.8)
- added R3: 0R_1608M, Applidyne_Resistor:RESC1608X50N, B.Cu at (139.7, 125.2)
- added R4: 0R_1608M, Applidyne_Resistor:RESC1608X50N, B.Cu at (139.6, 126.8)
- moved P0 51.6 mm to (92.5, 110.0), turned to 270 degrees
- moved P1 37.0 mm to (100.0, 100.0)
- moved P2 36.0 mm to (100.0, 110.0)
- moved P3 35.1 mm to (100.0, 120.0)
- moved P4 34.1 mm to (100.0, 130.0)
Connections:
- P1 pad P10: Net-(P1-PadP10) -> GND
- P1 pad P12: Net-(P1-PadP12) -> GND
- P1 pad P13: Net-(P1-PadP13) -> +12V
- P1 pad P14: Net-(P1-PadP14) -> +12V
- P1 pad P15: Net-(P1-PadP15) -> +12V
- P1 pad P4: Net-(P1-PadP4) -> GND
- P1 pad P5: Net-(P1-PadP5) -> GND
- P1 pad P6: Net-(P1-PadP6) -> GND
- P1 pad P7: Net-(P1-PadP7) -> +5V
- P1 pad P8: Net-(P1-PadP8) -> +5V
- P1 pad P9: Net-(P1-PadP9) -> +5V
- P1 pad S1: Net-(P1-PadS1) -> GND
- P1 pad S4: Net-(P1-PadS1) -> GND
- P1 pad S7: Net-(P1-PadS1) -> GND
- P2 pad P10: Net-(P2-PadP10) -> GND
- P2 pad P12: Net-(P2-PadP12) -> GND
- P2 pad P13: Net-(P2-PadP13) -> +12V
- P2 pad P14: Net-(P2-PadP14) -> +12V
- P2 pad P15: Net-(P2-PadP15) -> +12V
- P2 pad P4: Net-(P2-PadP4) -> GND
- P2 pad P5: Net-(P2-PadP5) -> GND
- P2 pad P6: Net-(P2-PadP6) -> GND
- P2 pad P7: Net-(P2-PadP7) -> +5V
- P2 pad P8: Net-(P2-PadP8) -> +5V
- P2 pad P9: Net-(P2-PadP9) -> +5V
- P2 pad S1: Net-(P2-PadS1) -> GND
- P2 pad S4: Net-(P2-PadS1) -> GND
- P2 pad S7: Net-(P2-PadS1) -> GND
- P3 pad P10: Net-(P3-PadP10) -> GND
- P3 pad P12: Net-(P3-PadP12) -> GND
- P3 pad P13: Net-(P3-PadP13) -> +12V
- P3 pad P14: Net-(P3-PadP14) -> +12V
- P3 pad P15: Net-(P3-PadP15) -> +12V
- P3 pad P4: Net-(P3-PadP4) -> GND
- P3 pad P5: Net-(P3-PadP5) -> GND
- P3 pad P6: Net-(P3-PadP6) -> GND
- P3 pad P7: Net-(P3-PadP7) -> +5V
- P3 pad P8: Net-(P3-PadP8) -> +5V
- P3 pad P9: Net-(P3-PadP9) -> +5V
- P3 pad S1: Net-(P3-PadS1) -> GND
- P3 pad S4: Net-(P3-PadS1) -> GND
- P3 pad S7: Net-(P3-PadS1) -> GND
- P4 pad P10: Net-(P4-PadP10) -> GND
- P4 pad P12: Net-(P4-PadP12) -> GND
- P4 pad P13: Net-(P4-PadP13) -> +12V
- P4 pad P14: Net-(P4-PadP14) -> +12V
- P4 pad P15: Net-(P4-PadP15) -> +12V
- P4 pad P4: Net-(P4-PadP4) -> GND
- P4 pad P5: Net-(P4-PadP5) -> GND
- P4 pad P6: Net-(P4-PadP6) -> GND
- P4 pad P7: Net-(P4-PadP7) -> +5V
- P4 pad P8: Net-(P4-PadP8) -> +5V
- P4 pad P9: Net-(P4-PadP9) -> +5V
- P4 pad S1: Net-(P4-PadS1) -> GND
- P4 pad S4: Net-(P4-PadS1) -> GND
- P4 pad S7: Net-(P4-PadS1) -> GND
Routing:
- net /RX0-: track 0.00 -> 34.6 mm
- net /TX3-: track 0.00 -> 32.4 mm
- net /TX3+: track 0.00 -> 31.6 mm
- net /TX0-: track 0.00 -> 30.8 mm
- net /RX0+: track 0.00 -> 30.8 mm
- net /RX3-: track 0.00 -> 28.2 mm
- net /RX3+: track 0.00 -> 27.4 mm
- net /TX0+: track 0.00 -> 27.2 mm
- net /TX1+: track 0.00 -> 24.9 mm, vias 0 -> 1
- net /TX2-: track 0.00 -> 24.7 mm, vias 0 -> 1
- net /TX1-: track 0.00 -> 24.1 mm, vias 0 -> 1
- net /TX2+: track 0.00 -> 23.5 mm, vias 0 -> 1
- net /RX2-: track 0.00 -> 21.1 mm
- net /RX2+: track 0.00 -> 20.2 mm
- net /RX1-: track 0.00 -> 19.1 mm
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- added copper zone on B.Cu, net +12V
- added copper zone on F.Cu, net +5V
- added copper zone on In2.Cu, net GND
Other:
- board outline added: 57.5 x 40 mm
- board text added: "12V"
- board text added: "5V"
- board text added: "GND"
- board text added: "OCLINK4i SATA"
- board text added: "SATA1"
- board text added: "SATA2"
- board text added: "SATA3"

Commit message: Continued routing/layout
Most pours done
Parts:
- moved R3 0.66 mm to (139.0, 125.2)
- moved R4 0.60 mm to (139.0, 126.8)
- moved C5 0.20 mm to (128.8, 105.8)
- moved C6 0.20 mm to (128.8, 116.0)
- moved C7 0.20 mm to (128.8, 126.0)
- moved R1 0.20 mm to (139.0, 105.2)
- moved R2 0.20 mm to (139.0, 106.8)
Routing:
- net GND: track 0.00 -> 110.5 mm, vias 0 -> 53
- net +12V: track 0.00 -> 19.7 mm
- net +5V: track 0.00 -> 19.4 mm
- net /RX0-: track 34.6 -> 17.1 mm
- net Net-(P3-PadP11): track 0.00 -> 12.6 mm, vias 0 -> 1
- net Net-(P1-PadP11): track 0.00 -> 12.5 mm, vias 0 -> 1
- net /RX0+: track 30.8 -> 19.6 mm
- net Net-(P4-PadP11): track 0.00 -> 10.9 mm, vias 0 -> 1
- net Net-(P2-PadP11): track 0.00 -> 10.8 mm, vias 0 -> 1
- net /TX3+: track 31.6 -> 30.5 mm
- net /TX3-: track 32.4 -> 31.3 mm
- net /TX0-: track 30.8 -> 29.8 mm
- net /TX0+: track 27.2 -> 26.2 mm
- net /RX3+: track 27.4 -> 26.5 mm
- net /RX3-: track 28.2 -> 27.4 mm
- added copper zone on B.Cu, net +5V
- added copper zone on In1.Cu, net +5V
- added copper zone on B.Cu, net GND
Other:
- outline, holes or cut-outs redrawn
- board text added: "OCCULINK 4i 4x SATA BACKPLANE"
- board text added: "S.RAPSON '21"
- board text added: "SATA4"
- board text removed: "OCLINK4i SATA"

Commit message: Diff pair skew tuning
Routing:
- net /TX0+: track 26.2 -> 30.7 mm
- net /RX0-: track 17.1 -> 19.6 mm
- net /TX2+: track 23.5 -> 25.4 mm
- net GND: track 110.5 -> 111.4 mm
- net /TX0-: track 29.8 -> 30.7 mm
- net /TX3+: track 30.5 -> 31.4 mm
- net /RX1+: track 18.4 -> 19.2 mm
- net /RX2+: track 20.1 -> 21.0 mm
- net /TX1-: track 24.1 -> 24.9 mm
- net /RX3+: track 26.5 -> 27.2 mm
